File: doc/Anzeige_Simon10/Anzeige_Simon.kicad_pcb (KiCad board)
At the start: 2 copper layers, 50 x 37 mm, 20 parts, among them J1 I2C, J2 Daten, J3 MoGND, J4 Vcc, J5 AnzByte, U1 74HC688, U2 PCF8574P, U3 SFH617

Commit message: 
Parts:
- added TP1, TP2: TP-GND, TestPoint:TestPoint_Keystone_5019_Miniature, F.Cu at (81.0, 52.0)

Commit message: update files
new testpoints
Parts:
- TP1: value TP-GND -> TP Up; footprint TestPoint:TestPoint_Keystone_5019_Miniature -> Connector_Wire:SolderWirePad_1x01_SMD_1x2mm
- TP2: value TP-GND -> TP Down; footprint TestPoint:TestPoint_Keystone_5019_Miniature -> Connector_Wire:SolderWirePad_1x01_SMD_1x2mm; moved to B.Cu
- moved TP1 1.58 mm to (82.5, 51.5), turned to 90 degrees
- moved TP2 1.58 mm to (82.5, 51.5), turned to -90 degrees

Commit message: update files
add holes
Parts:
- removed TP1: TP Up, Connector_Wire:SolderWirePad_1x01_SMD_1x2mm
- removed TP2: TP Down, Connector_Wire:SolderWirePad_1x01_SMD_1x2mm
- added GND1: GND TP, Connector_Wire:SolderWirePad_1x01_SMD_1x2mm, F.Cu at (82.5, 82.5)
- added GND2: GND TP, Connector_Wire:SolderWirePad_1x01_SMD_1x2mm, B.Cu at (82.5, 82.5)
- added H1: Befestigung, MountingHole:MountingHole_3.2mm_M3_ISO14580, F.Cu at (81.0, 51.0)
- added H2: Befestigung, MountingHole:MountingHole_3.2mm_M3_ISO14580, F.Cu at (60.9, 51.0)
- added H3: Befestigung, MountingHole:MountingHole_3.2mm_M3_ISO14580, F.Cu at (38.0, 81.0)
- moved R7 8.00 mm to (49.5, 80.0)
- moved R8 1.75 mm to (52.2, 80.0)
- moved J4 1.64 mm to (78.0, 79.5)
- moved R1 1.00 mm to (55.5, 54.5)
- moved J3 0.50 mm to (40.0, 51.8)
- moved U3 0.50 mm to (52.3, 54.3)
- moved J2 0.48 mm to (40.0, 61.0)
Routing:
- net +5V: track 118.3 -> 111.8 mm
- net Net-(U1-P=R): track 8.31 -> 8.84 mm
- net Net-(J5-Pin_8): track 30.0 -> 29.5 mm
- net Net-(R1-Pad2): track 2.79 -> 2.29 mm
- net GND: vias 23 -> 24

Commit message: Update files
Parts:
- JP1, JP2, JP3: value ~ -> Jumper_3_Open; footprint Jumper:SolderJumper-2_P1.3mm_Open_RoundedPad1.0x1.5mm -> Jumper:SolderJumper-3_P1.3mm_Open_RoundedPad1.0x1.5mm
- R1: value 330 -> 220
- moved JP2 0.33 mm to (70.5, 56.5), turned to 90 degrees
- moved JP3 0.33 mm to (73.5, 56.5), turned to 90 degrees
- moved JP1 0.31 mm to (67.3, 56.5), turned to 90 degrees
- moved R4 0.25 mm to (67.3, 51.1)
- moved R5 0.25 mm to (70.5, 51.1)
- moved R6 0.25 mm to (73.5, 51.1)
- renumbered R6 to R4, R4 to R6
Connections:
- net +5V renamed Vcc
- JP1 pad 1: Net-(JP1-A) -> GND
- JP1 pad 2: Net-(JP1-B) -> A0
- JP2 pad 1: Net-(JP2-A) -> GND
- JP2 pad 2: Net-(JP2-B) -> A1
- JP3 pad 1: Net-(JP3-A) -> GND
- JP3 pad 2: Net-(JP3-B) -> A2
- R4 pad 2: Net-(JP1-A) -> Net-(JP1-B)
- R5 pad 2: Net-(JP2-A) -> Net-(JP2-B)
- R6 pad 2: Net-(JP3-A) -> Net-(JP3-B)
- U2 pad 1: Net-(JP1-B) -> A0
- U2 pad 2: Net-(JP2-B) -> A1
- U2 pad 3: Net-(JP3-B) -> A2
Routing:
- net A2: track 0.00 -> 13.6 mm
- net Net-(JP3-B): track 12.9 -> 3.10 mm
- net A1: track 0.00 -> 9.76 mm
- net A0: track 0.00 -> 7.04 mm
- net Net-(JP2-B): track 9.77 -> 3.10 mm
- net Net-(JP1-B): track 5.02 -> 0.00 mm
- net Net-(JP3-A): track 3.26 -> 0.00 mm
- net Net-(JP2-A): track 3.26 -> 0.00 mm
- net Net-(JP1-A): track 3.20 -> 0.00 mm
- net Vcc: track 111.8 -> 112.8 mm
- net GND: vias 24 -> 23

Commit message: Add files via upload
Parts:
- JP1, JP2, JP3: value Jumper_3_Open -> ~; footprint Jumper:SolderJumper-3_P1.3mm_Open_RoundedPad1.0x1.5mm -> Jumper:SolderJumper-2_P1.3mm_Open_RoundedPad1.0x1.5mm
- R1: value 220 -> 330
- moved JP2 0.33 mm to (70.3, 56.2), turned to -90 degrees
- moved JP3 0.33 mm to (73.3, 56.2), turned to -90 degrees
- moved JP1 0.31 mm to (67.3, 56.2), turned to -90 degrees
- moved R4 0.25 mm to (73.5, 51.4)
- moved R5 0.25 mm to (70.5, 51.4)
- moved R6 0.25 mm to (67.3, 51.4)
- renumbered R6 to R4, R4 to R6
Connections:
- net A0 renamed Net-(JP1-B)
- net A1 renamed Net-(JP2-B)
- net A2 renamed Net-(JP3-B)
- net Vcc renamed +5V
- JP1 pad 1: GND -> Net-(JP1-A)
- JP2 pad 1: GND -> Net-(JP2-A)
- JP3 pad 1: GND -> Net-(JP3-A)
- R4 pad 2: Net-(JP3-B) (its old number) -> Net-(JP3-A)
- R5 pad 2: Net-(JP2-B) (its old number) -> Net-(JP2-A)
- R6 pad 2: Net-(JP1-B) (its old number) -> Net-(JP1-A)
Routing:
- net Net-(JP3-A): track 0.00 -> 3.26 mm
- net Net-(JP2-A): track 0.00 -> 3.26 mm
- net Net-(JP1-A): track 0.00 -> 3.20 mm
- net Net-(JP3-B) (its old number): track 3.10 -> 0.00 mm
- net Net-(JP2-B) (its old number): track 3.10 -> 0.00 mm
- net Net-(JP1-B): track 7.04 -> 5.02 mm
- net +5V: track 112.8 -> 111.8 mm
- net Net-(JP3-B): track 13.6 -> 12.9 mm
- net GND: vias 23 -> 24
