File: doc/Anzeige_Simon10/Anzeige_Simon.kicad_sch (KiCad schematic)
At the start: 20 parts, among them J1 I2C, J2 Daten, J3 MoGND, J4 Vcc, J5 AnzByte, U1 74HC688, U2 PCF8574P, U3 SFH617

Commit message: 
Parts:
- added TP1, TP2: TP-GND, TestPoint:TestPoint_Keystone_5019_Miniature, symbol Connector:TestPoint_Square
Connections:
- net GND: now also TP1.1, TP2.1

Commit message: update files
new testpoints
Parts:
- removed TP1, TP2: TP-GND, TestPoint:TestPoint_Keystone_5019_Miniature, symbol Connector:TestPoint_Square
- added TP1: TP Up, Connector_Wire:SolderWirePad_1x01_SMD_1x2mm, symbol Connector:TestPoint
- added TP2: TP Down, Connector_Wire:SolderWirePad_1x01_SMD_1x2mm, symbol Connector:TestPoint
Connections:
- net GND: now also TP1.1, TP2.1

Commit message: update files
add holes
Parts:
- added H1, H2, H3: Befestigung, MountingHole:MountingHole_3.2mm_M3_ISO14580, symbol Mechanical:MountingHole
- GND1: renamed from TP1; value TP Up -> GND TP
- GND2: renamed from TP2; value TP Down -> GND TP
Changed lines of the file:
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@@
+	)
+	(symbol
+		(lib_id "Mechanical:MountingHole")
+		(at 158.75 95.25 0)
+		(unit 1)
+		(body_style 1)
+		(exclude_from_sim no)
+		(in_bom no)
+		(on_board yes)
+		(in_pos_files yes)
+		(dnp no)
+		(fields_autoplaced yes)
+		(property "Reference" "H2"
+			(at 161.29 93.9799 0)
+			(show_name no)
+			(do_not_autoplace no)
+			(effects
+				(font
+					(size 1.27 1.27)
+				)
+				(justify left)
+			)
+		)
+		(property "Value" "Befestigung"
+			(at 161.29 96.5199 0)
+			(show_name no)
+			(do_not_autoplace no)
+			(effects
+				(font
+					(size 1.27 1.27)
+				)
+				(justify left)
+			)
+		)
+		(property "Footprint" "MountingHole:MountingHole_3.2mm_M3_ISO14580"
+			(at 158.75 95.25 0)
+			(hide yes)
+			(show_name no)
+			(do_not_autoplace no)
+			(effects
+				(font
+					(size 1.27 1.27)
+				)
+			)
+		)
+		(property "Datasheet" ""
+			(at 158.75 95.25 0)
+			(hide yes)
+			(show_name no)
+			(do_not_autoplace no)
+			(effects
+				(font
+					(size 1.27 1.27)
+				)
+			)
+		)
+		(property "Description" "Mounting Hole without connection"
+			(at 158.75 95.25 0)
+			(hide yes)
+			(show_name no)
+			(do_not_autoplace no)
+			(effects
+				(font
+					(size 1.27 1.27)
+				)
+			)
+		)
+		(instances
+			(project "Anzeige_Simon"
+				(path "/faaf0afd-d19d-41db-9e1b-72a0c1b6f023"
+					(reference "H2")
+					(unit 1)
+				)
+			)
+		)
 	)
 	(symbol
@@
 		(in_pos_files yes)
 		(dnp no)
-		(property "Reference" "TP2"
+		(property "Reference" "GND2"
 			(at 164.084 78.232 0)
 			(show_name no)
@@
 			)
 		)
-		(property "Value" "TP Down"
+		(property "Value" "GND TP"
 			(at 165.608 80.772 0)
 			(show_name no)
@@
 			(project "Anzeige_Simon"
 				(path "/faaf0afd-d19d-41db-9e1b-72a0c1b6f023"
-					(reference "TP2")
+					(reference "GND2")
 					(unit 1)
 				)
@@
 		(in_pos_files yes)
 		(dnp no)
-		(property "Reference" "TP1"
+		(property "Reference" "GND1"
 			(at 152.654 78.232 0)
 			(show_name no)
@@
 			)
 		)
-		(property "Value" "TP Up"
+		(property "Value" "GND TP"
 			(at 154.178 80.772 0)
 			(show_name no)
@@
 			(project "Anzeige_Simon"
 				(path "/faaf0afd-d19d-41db-9e1b-72a0c1b6f023"
-					(reference "TP1")
+					(reference "GND1")
 					(unit 1)
 				)
@@
 	)
 	(symbol
+		(lib_id "Mechanical:MountingHole")
+		(at 88.9 110.49 0)
+		(unit 1)
+		(body_style 1)
+		(exclude_from_sim no)
+		(in_bom no)
+		(on_board yes)
+		(in_pos_files yes)
+		(dnp no)
+		(fields_autoplaced yes)
+		(property "Reference" "H3"
+			(at 91.44 109.2199 0)
+			(show_name no)
+			(do_not_autoplace no)
+			(effects
+				(font
+					(size 1.27 1.27)
+				)
+				(justify left)
+			)
+		)
+		(property "Value" "Befestigung"
+			(at 91.44 111.7599 0)
+			(show_name no)
+			(do_not_autoplace no)
+			(effects
+				(font
+					(size 1.27 1.27)
+				)
+				(justify left)
+			)
+		)
+		(property "Footprint" "MountingHole:MountingHole_3.2mm_M3_ISO14580"
+			(at 88.9 110.49 0)
+			(hide yes)
+			(show_name no)
+			(do_not_autoplace no)
+			(effects
+				(font
+					(size 1.27 1.27)
+				)
+			)
+		)
+		(property "Datasheet" ""
+			(at 88.9 110.49 0)
+			(hide yes)
+			(show_name no)
+			(do_not_autoplace no)
+			(effects
+				(font
+					(size 1.27 1.27)
+				)
+			)
+		)
+		(property "Description" "Mounting Hole without connection"
+			(at 88.9 110.49 0)
+			(hide yes)
+			(show_name no)
+			(do_not_autoplace no)
+			(effects
+				(font
+					(size 1.27 1.27)
+				)
+			)
+		)
+		(instances
+			(project "Anzeige_Simon"
+				(path "/faaf0afd-d19d-41db-9e1b-72a0c1b6f023"
+					(reference "H3")
+					(unit 1)
+				)
+			)
+		)
+	)
+	(symbol
 		(lib_id "Device:R")
 		(at 72.39 49.53 0)
@@
 					(unit 1)
 				)
+			)
+		)
+	)
+	(symbol
+		(lib_id "Mechanical:MountingHole")
+		(at 114.3 50.8 0)
+		(unit 1)
+		(body_style 1)
+		(exclude_from_sim no)
+		(in_bom no)
+		(on_board yes)
+		(in_pos_files yes)
+		(dnp no)
+		(fields_autoplaced yes)
+		(property "Reference" "H1"
+			(at 116.84 49.5299 0)
+			(show_name no)
+			(do_not_autoplace no)
+			(effects
+				(font
+					(size 1.27 1.27)
+				)
+				(justify left)
+			)
+		)
+		(property "Value" "Befestigung"
+			(at 116.84 52.0699 0)
+			(show_name no)
+			(do_not_autoplace no)
+			(effects
+				(font
+					(size 1.27 1.27)
+				)
+				(justify left)
+			)
+		)
+		(property "Footprint" "MountingHole:MountingHole_3.2mm_M3_ISO14580"
+			(at 114.3 50.8 0)
+			(hide yes)
+			(show_name no)
+			(do_not_autoplace no)
+			(effects
+				(font
+					(size 1.27 1.27)
+				)
+			)
+		)
+		(property "Datasheet" ""
+			(at 114.3 50.8 0)
+			(hide yes)
+			(show_name no)
+			(do_not_autoplace no)
+			(effects
+				(font
+					(size 1.27 1.27)
+				)
+			)
+		)
+		(property "Description" "Mounting Hole without connection"
+			(at 114.3 50.8 0)
+			(hide yes)
+			(show_name no)
+			(do_not_autoplace no)
+			(effects
+				(font
+					(size 1.27 1.27)
+				)
+			)
+		)
+		(instances
+			(project "Anzeige_Simon"
+				(path "/faaf0afd-d19d-41db-9e1b-72a0c1b6f023"
+					(reference "H1")
+					(unit 1)
+				)

Commit message: Update files
Parts:
- removed JP1, JP2, JP3: (no value), Jumper:SolderJumper-2_P1.3mm_Open_RoundedPad1.0x1.5mm, symbol Jumper:Jumper_2_Open
- added JP1, JP2, JP3: Jumper_3_Open, Jumper:SolderJumper-3_P1.3mm_Open_RoundedPad1.0x1.5mm, symbol Jumper:Jumper_3_Open
- R1: value 330 -> 220
- renumbered R6 to R4, R4 to R6
Connections:
- net GND: now also JP1.1 (A), JP2.1 (A), JP3.1 (A)
- net at R5.2: now also JP2.3 (B)
- net A1: now reaches U2.2 (A1)
- net A1: now also JP2.2 (C)
- net at R4.2: now also JP1.3 (B)
- net A0: now reaches U2.1 (A0)
- net A0: now also JP1.2 (C)
- net A2: now reaches U2.3 (A2)
- net A2: now also JP3.2 (C)
- net at R6.2: now also JP3.3 (B)
- net +5V renamed Vcc
Other:
- moved on the sheet: GND1, GND2, H1, H2, H3, J1, J2, J3, J4, J5, R1, R2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

Commit message: Add files via upload
Parts:
- removed JP1, JP2, JP3: Jumper_3_Open, Jumper:SolderJumper-3_P1.3mm_Open_RoundedPad1.0x1.5mm, symbol Jumper:Jumper_3_Open
- added JP1, JP2, JP3: (no value), Jumper:SolderJumper-2_P1.3mm_Open_RoundedPad1.0x1.5mm, symbol Jumper:Jumper_2_Open
- R1: value 220 -> 330
- renumbered R6 to R4, R4 to R6
Connections:
- net at R5.2: now also JP2.1 (A)
- net at R4.2: now also JP3.1 (A)
- net at R6.2: now also JP1.1 (A)
- net A0: no longer names the net of U2.1 (A0)
- net A0: now also JP1.2 (B)
- net A1: no longer names the net of U2.2 (A1)
- net A1: now also JP2.2 (B)
- net A2: no longer names the net of U2.3 (A2)
- net A2: now also JP3.2 (B)
- net Vcc renamed +5V
Other:
- moved on the sheet: GND1, GND2, H1, H2, H3, J1, J2, J3, J4, J5, R1, R2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
